File: Hardware/Electrical Components/Module - Power/Power module.sch (EAGLE design)
At the start: 97 parts

Commit message: Updates
Updated eDNA Eagle Library
Update OpenSPower7.2 BOM
Add OpenSPower 7.2 ReadMe
Add picture for FlowSensor
General clean up
Parts:
- removed C2: 100nF, adafruit:C-US050-024X044
Connections:
- net +5V: no longer C2.1
- net GND: no longer C2.2
Changed lines of the file:
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@@
 <part name="GND1" library="SparkFun-PowerSymbols" library_urn="urn:adsk.eagle:library:530" deviceset="GND" device=""/>
 <part name="+3V1" library="supply1" library_urn="urn:adsk.eagle:library:371" deviceset="+3V3" device=""/>
-<part name="C2" library="adafruit" library_urn="urn:adsk.eagle:library:420" deviceset="C-US" device="050-024X044" package3d_urn="urn:adsk.eagle:package:6240356/1" value="100nF"/>
 <part name="P+1" library="supply1" library_urn="urn:adsk.eagle:library:371" deviceset="+5V" device=""/>
 <part name="GND2" library="SparkFun-PowerSymbols" library_urn="urn:adsk.eagle:library:530" deviceset="GND" device=""/>
@@
 <attribute name="VALUE" x="-119.38" y="76.2" size="1.778" layer="96" rot="R90"/>
 </instance>
-<instance part="C2" gate="G$1" x="-22.86" y="76.2" smashed="yes" rot="R270">
-<attribute name="NAME" x="-22.225" y="75.184" size="1.778" layer="95" rot="R270"/>
-<attribute name="VALUE" x="-24.511" y="72.644" size="1.778" layer="96" rot="R270"/>
-</instance>
 <instance part="P+1" gate="1" x="-20.32" y="81.28" smashed="yes">
 <attribute name="VALUE" x="-22.86" y="81.28" size="1.778" layer="96" rot="R90"/>
@@
 <pinref part="B1" gate="G$1" pin="GND@2"/>
 <wire x1="-50.8" y1="76.2" x2="-27.94" y2="76.2" width="0.1524" layer="91"/>
-<pinref part="C2" gate="G$1" pin="2"/>
 <pinref part="GND2" gate="1" pin="GND"/>
-<junction x="-27.94" y="76.2"/>
 </segment>
 <segment>
@@
 </segment>
 <segment>
-<pinref part="C2" gate="G$1" pin="1"/>
-<wire x1="-20.32" y1="76.2" x2="-20.32" y2="78.74" width="0.1524" layer="91"/>
 <pinref part="P+1" gate="1" pin="+5V"/>
 <pinref part="B1" gate="G$1" pin="HV"/>
 <wire x1="-20.32" y1="78.74" x2="-50.8" y2="78.74" width="0.1524" layer="91"/>
-<junction x="-20.32" y="78.74"/>
-</segment>
-<segment>
+</segment>
+<segment>
